File: Schematic/fpv-diversity.sch (EAGLE design)
At the start: 32 parts, among them U1 LM1881M/NOPB, U2 LM1881M/NOPB, U3 LM1881M/NOPB, U4 MAX4545CAP+

Commit message: PCB updates
Parts:
- removed 5V, VID1, VID2, VID3, VOUTDIV: (no value), pinhead:PINHD-1X2
- added 12V, OUT1, OUT2, RX1, RX2, RX3: (no value), pinhead:PINHD-1X2
- added C11: 1nF, rcl:C-USC0805
- added C12, C13, C14, C16, C17, C18: 100nF, rcl:C-USC0805
- added C15: 47uF, rcl:CPOL-USCT3528
- added C19: 10uF, rcl:CPOL-EUD
- added C20: 33uF, rcl:CPOL-EUD
- added C21: 4.7uF, rcl:CPOL-USCT3528
- added C22, C23: 470uF, rcl:CPOL-USCT3528
- added PWR: (no value), led:LEDCHIP-LED0805
- added R10, R14: 1K, rcl:R-US_R1206
- added R11, R15: 4.7K, rcl:R-US_R1206
- added R12: 680K, rcl:R-US_R1206
- added R13, R17, R18: 75, rcl:R-US_R1206
- added R16: 470, rcl:R-US_R1206
- added R19, R20, R21, R22: 499, rcl:R-US_R1206
- added U5: LT6206CMS8PBF, LT6206CMS8PBF:LT6206CMS8PBF
- added U6: LM1117IMP-5.0-NOPB, LM1117IMP-5.0-NOPB:LM1117IMP-5.0-NOPB
- C1, C10, C2, C3, C6, C9: device rcl:C-USC0402 -> rcl:C-USC0805
- C4: value 1nF -> 47uF; device rcl:C-USC0402 -> rcl:CPOL-USCT3528
- C5: value 100nF -> 1nF; device rcl:C-USC0402 -> rcl:C-USC0805
- C7: value 1nF -> 100nF; device rcl:C-USC0402 -> rcl:C-USC0805
- C8: value 100nF -> 47uF; device rcl:C-USC0402 -> rcl:CPOL-USCT3528
- R1, R3, R4, R5, R6, R9: device rcl:R-US_R0603 -> rcl:R-US_R1206
- R2: value 680K -> 75; device rcl:R-US_R0603 -> rcl:R-US_R1206
- R7: value 75 -> 1K; device rcl:R-US_R0603 -> rcl:R-US_R1206
- R8: value 75 -> 4.7K; device rcl:R-US_R0603 -> rcl:R-US_R1206
Connections:
- removed net 1N1: U$1.D1
- removed net N$6: C8.2, U3.COMPOSITESYNCIN
- removed net VOUT: U4.COM1, U4.COM2, U4.COM3, VOUTDIV.1
- new net 5V: C10.1, C14.1, C16.1, C17.1, C18.1, C20.+, C21.+, C9.1, R11.2, R15.2, R16.2, R8.2, U$1.5V, U1.VCC, U2.VCC, U3.VCC, U4.V+, U5.V+, U6.OUT
- new net N$10: C13.1, R12.2, U1.RSET
- new net N$11: C12.2, U1.COMPOSITESYNCIN
- new net N$12: R19.1, R20.2, U5.-INA
- new net N$13: R18.2, R21.1, U5.OUTB
- new net N$14: R21.2, R22.1, U5.-INB
- new net N$15: R17.1, R20.1, U5.OUTA
- new net N$16: C22.+, R18.1
- new net N$17: C23.+, R17.2
- new net PRE-VOUT: U4.COM1, U4.COM2, U4.COM3, U5.+INA, U5.+INB
- new net VID1: C12.1, C15.-, R13.2, RX1.1
- new net VID2: C2.1, C4.-, R2.2, RX2.1
- new net VID3: C6.1, C8.-, R9.2, RX3.1
- new net VOUT1: C22.-, OUT1.1
- new net VOUT2: C23.-, OUT2.1
- net BPOUT1: now also C11.1; no longer C1.1
- net BPOUT2: now also C1.1; no longer C4.1
- net BPOUT3: now also C5.1; no longer C7.1
- net GND: now also 12V.2, C11.2, C13.2, C14.2, C16.2, C17.2, C18.2, C19.-, C20.-, C21.-, C5.2, OUT1.2, OUT2.2, PWR.C, R10.1, R12.1, R13.1, R14.1, R19.2, R22.2, RX1.2, RX2.2, RX3.2, U5.V-, U6.GND; no longer 5V.2, C4.2, C6.2, R8.1, VID1.2, VID2.2, VID3.2, VOUTDIV.2
- net IN1: now also U$1.D1
- net N$1: now also C7.1, R3.2, U3.RSET; no longer C2.2, U1.COMPOSITESYNCIN
- net N$2: now also C3.1, R1.2; no longer C6.1, R2.2
- net N$3: now also C2.2, U2.COMPOSITESYNCIN; no longer C3.1, R1.2, U1.RSET
- net N$4: now also PWR.A, R16.1; no longer C5.2, U2.COMPOSITESYNCIN
- net N$5: now also C6.2, U3.COMPOSITESYNCIN; no longer C9.1, R3.2, U3.RSET
- net N01: now also C15.+, R14.2, R15.1; no longer C2.1, R7.2, VID1.1
- net N02: now also C4.+, R7.2, R8.1; no longer C5.1, R8.2, VID2.1
- net N03: now also C8.+, R10.2, R11.1; no longer C8.1, R9.2, VID3.1
- net VCC: now also 12V.1, C19.+, U6.IN; no longer 5V.1, C10.1, U$1.5V, U1.VCC, U2.VCC, U3.VCC, U4.V+
Other:
- moved on the sheet: C1, C10, C2, C3, C5, C6, C7, C9, LED1, LED2, LED3, R1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

Commit message: .brd cleanup
Parts:
- C15, C4, C8: device rcl:CPOL-USCT3528 -> rcl:CPOL-USCT3216
- C22, C23: device rcl:CPOL-USCT3528 -> rcl:CPOL-USCT7343
Changed lines of the file:
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@@
 <part name="GND4" library="supply1" library_urn="urn:adsk.eagle:library:371" deviceset="GND" device=""/>
 <part name="U2" library="LM1881M_NOPB" deviceset="LM1881M/NOPB" device="" package3d_urn="urn:adsk.eagle:package:18494142/1"/>
-<part name="C4" library="rcl" library_urn="urn:adsk.eagle:library:334" deviceset="CPOL-US" device="CT3528" package3d_urn="urn:adsk.eagle:package:23325/2" value="47uF"/>
+<part name="C4" library="rcl" library_urn="urn:adsk.eagle:library:334" deviceset="CPOL-US" device="CT3216" package3d_urn="urn:adsk.eagle:package:23327/2" value="47uF"/>
 <part name="R7" library="rcl" library_urn="urn:adsk.eagle:library:334" deviceset="R-US_" device="R1206" package3d_urn="urn:adsk.eagle:package:23540/2" value="1K"/>
 <part name="GND5" library="supply1" library_urn="urn:adsk.eagle:library:371" deviceset="GND" device=""/>
@@
 <part name="GND9" library="supply1" library_urn="urn:adsk.eagle:library:371" deviceset="GND" device=""/>
 <part name="U3" library="LM1881M_NOPB" deviceset="LM1881M/NOPB" device="" package3d_urn="urn:adsk.eagle:package:18494142/1"/>
-<part name="C8" library="rcl" library_urn="urn:adsk.eagle:library:334" deviceset="CPOL-US" device="CT3528" package3d_urn="urn:adsk.eagle:package:23325/2" value="47uF"/>
+<part name="C8" library="rcl" library_urn="urn:adsk.eagle:library:334" deviceset="CPOL-US" device="CT3216" package3d_urn="urn:adsk.eagle:package:23327/2" value="47uF"/>
 <part name="R10" library="rcl" library_urn="urn:adsk.eagle:library:334" deviceset="R-US_" device="R1206" package3d_urn="urn:adsk.eagle:package:23540/2" value="1K"/>
 <part name="GND12" library="supply1" library_urn="urn:adsk.eagle:library:371" deviceset="GND" device=""/>
@@
 <part name="GND21" library="supply1" library_urn="urn:adsk.eagle:library:371" deviceset="GND" device=""/>
 <part name="U1" library="LM1881M_NOPB" deviceset="LM1881M/NOPB" device="" package3d_urn="urn:adsk.eagle:package:18494142/1"/>
-<part name="C15" library="rcl" library_urn="urn:adsk.eagle:library:334" deviceset="CPOL-US" device="CT3528" package3d_urn="urn:adsk.eagle:package:23325/2" value="47uF"/>
+<part name="C15" library="rcl" library_urn="urn:adsk.eagle:library:334" deviceset="CPOL-US" device="CT3216" package3d_urn="urn:adsk.eagle:package:23327/2" value="47uF"/>
 <part name="R14" library="rcl" library_urn="urn:adsk.eagle:library:334" deviceset="R-US_" device="R1206" package3d_urn="urn:adsk.eagle:package:23540/2" value="1K"/>
 <part name="GND23" library="supply1" library_urn="urn:adsk.eagle:library:371" deviceset="GND" device=""/>
@@
 <part name="C21" library="rcl" library_urn="urn:adsk.eagle:library:334" deviceset="CPOL-US" device="CT3528" package3d_urn="urn:adsk.eagle:package:23325/2" value="4.7uF"/>
 <part name="GND34" library="supply1" library_urn="urn:adsk.eagle:library:371" deviceset="GND" device=""/>
-<part name="C22" library="rcl" library_urn="urn:adsk.eagle:library:334" deviceset="CPOL-US" device="CT3528" package3d_urn="urn:adsk.eagle:package:23325/2" value="470uF"/>
-<part name="C23" library="rcl" library_urn="urn:adsk.eagle:library:334" deviceset="CPOL-US" device="CT3528" package3d_urn="urn:adsk.eagle:package:23325/2" value="470uF"/>
+<part name="C22" library="rcl" library_urn="urn:adsk.eagle:library:334" deviceset="CPOL-US" device="CT7343" package3d_urn="urn:adsk.eagle:package:23304/2" value="470uF"/>
+<part name="C23" library="rcl" library_urn="urn:adsk.eagle:library:334" deviceset="CPOL-US" device="CT7343" package3d_urn="urn:adsk.eagle:package:23304/2" value="470uF"/>
 </parts>
 <sheets>

Commit message: Updates
Parts:
- C1, C11, C5: device rcl:C-USC0805 -> rcl:C-USC0603
- C19, C20: device rcl:CPOL-EUD -> rcl:CPOL-EUUD-4X5,8
- C22, C23: device rcl:CPOL-USCT7343 -> rcl:CPOL-USUD-6,3X7,7
- LED1, LED2, LED3, PWR: device led:LEDCHIP-LED0805 -> led:LEDCHIPLED_0603
- R16, R4, R5, R6: value 470 -> 120; device rcl:R-US_R1206 -> rcl:R-US_R0603

Commit message: Updates
Parts:
- added D1: (no value), diode:DIODE-DO-214AC
- C19, C20: device rcl:CPOL-EUUD-4X5,8 -> rcl:CPOL-EUD/7343-31W
- R1, R10, R11, R12, R14, R15, R17, R18, R3, R7, R8: device rcl:R-US_R1206 -> rcl:R-US_R0805
Connections:
- new net N$6: 12V.1, D1.A
- net VCC: now also D1.C; no longer 12V.1

Commit message: more updates
Parts:
- R13, R2, R9: device rcl:R-US_R1206 -> rcl:R-US_R0805
Changed lines of the file:
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@@
 <part name="C3" library="rcl" library_urn="urn:adsk.eagle:library:334" deviceset="C-US" device="C0805" package3d_urn="urn:adsk.eagle:package:23617/2" value="100nF"/>
 <part name="GND3" library="supply1" library_urn="urn:adsk.eagle:library:371" deviceset="GND" device=""/>
-<part name="R2" library="rcl" library_urn="urn:adsk.eagle:library:334" deviceset="R-US_" device="R1206" package3d_urn="urn:adsk.eagle:package:23540/2" value="75"/>
+<part name="R2" library="rcl" library_urn="urn:adsk.eagle:library:334" deviceset="R-US_" device="R0805" package3d_urn="urn:adsk.eagle:package:23553/2" value="75"/>
 <part name="GND4" library="supply1" library_urn="urn:adsk.eagle:library:371" deviceset="GND" device=""/>
 <part name="U2" library="LM1881M_NOPB" deviceset="LM1881M/NOPB" device="" package3d_urn="urn:adsk.eagle:package:18494142/1"/>
@@
 <part name="C7" library="rcl" library_urn="urn:adsk.eagle:library:334" deviceset="C-US" device="C0805" package3d_urn="urn:adsk.eagle:package:23617/2" value="100nF"/>
 <part name="GND8" library="supply1" library_urn="urn:adsk.eagle:library:371" deviceset="GND" device=""/>
-<part name="R9" library="rcl" library_urn="urn:adsk.eagle:library:334" deviceset="R-US_" device="R1206" package3d_urn="urn:adsk.eagle:package:23540/2" value="75"/>
+<part name="R9" library="rcl" library_urn="urn:adsk.eagle:library:334" deviceset="R-US_" device="R0805" package3d_urn="urn:adsk.eagle:package:23553/2" value="75"/>
 <part name="GND9" library="supply1" library_urn="urn:adsk.eagle:library:371" deviceset="GND" device=""/>
 <part name="U3" library="LM1881M_NOPB" deviceset="LM1881M/NOPB" device="" package3d_urn="urn:adsk.eagle:package:18494142/1"/>
@@
 <part name="C13" library="rcl" library_urn="urn:adsk.eagle:library:334" deviceset="C-US" device="C0805" package3d_urn="urn:adsk.eagle:package:23617/2" value="100nF"/>
 <part name="GND20" library="supply1" library_urn="urn:adsk.eagle:library:371" deviceset="GND" device=""/>
-<part name="R13" library="rcl" library_urn="urn:adsk.eagle:library:334" deviceset="R-US_" device="R1206" package3d_urn="urn:adsk.eagle:package:23540/2" value="75"/>
+<part name="R13" library="rcl" library_urn="urn:adsk.eagle:library:334" deviceset="R-US_" device="R0805" package3d_urn="urn:adsk.eagle:package:23553/2" value="75"/>
 <part name="GND21" library="supply1" library_urn="urn:adsk.eagle:library:371" deviceset="GND" device=""/>
 <part name="U1" library="LM1881M_NOPB" deviceset="LM1881M/NOPB" device="" package3d_urn="urn:adsk.eagle:package:18494142/1"/>

Commit message: Latest
Connections:
- net BPOUT2: now also U$1.D7; no longer U$1.D3
Changed lines of the file:
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@@
 <grid distance="0.1" unitdist="inch" unit="inch" style="lines" multiple="1" display="no" altdistance="0.01" altunitdist="inch" altunit="inch"/>
 <layers>
-<layer number="1" name="Top" color="4" fill="1" visible="yes" active="no"/>
-<layer number="2" name="Route2" color="16" fill="1" visible="yes" active="no"/>
-<layer number="3" name="Route3" color="17" fill="1" visible="yes" active="no"/>
-<layer number="4" name="Route4" color="18" fill="1" visible="yes" active="no"/>
-<layer number="5" name="Route5" color="19" fill="1" visible="yes" active="no"/>
-<layer number="6" name="Route6" color="25" fill="1" visible="yes" active="no"/>
-<layer number="7" name="Route7" color="26" fill="1" visible="yes" active="no"/>
-<layer number="8" name="Route8" color="27" fill="1" visible="yes" active="no"/>
-<layer number="9" name="Route9" color="28" fill="1" visible="yes" active="no"/>
-<layer number="10" name="Route10" color="29" fill="1" visible="yes" active="no"/>
-<layer number="11" name="Route11" color="30" fill="1" visible="yes" active="no"/>
-<layer number="12" name="Route12" color="20" fill="1" visible="yes" active="no"/>
-<layer number="13" name="Route13" color="21" fill="1" visible="yes" active="no"/>
-<layer number="14" name="Route14" color="22" fill="1" visible="yes" active="no"/>
-<layer number="15" name="Route15" color="23" fill="1" visible="yes" active="no"/>
-<layer number="16" name="Bottom" color="1" fill="1" visible="yes" active="no"/>
-<layer number="17" name="Pads" color="2" fill="1" visible="yes" active="no"/>
-<layer number="18" name="Vias" color="2" fill="1" visible="yes" active="no"/>
-<layer number="19" name="Unrouted" color="6" fill="1" visible="yes" active="no"/>
-<layer number="20" name="Dimension" color="24" fill="1" visible="yes" active="no"/>
-<layer number="21" name="tPlace" color="7" fill="1" visible="yes" active="no"/>
-<layer number="22" name="bPlace" color="7" fill="1" visible="yes" active="no"/>
-<layer number="23" name="tOrigins" color="15" fill="1" visible="yes" active="no"/>
-<layer number="24" name="bOrigins" color="15" fill="1" visible="yes" active="no"/>
-<layer number="25" name="tNames" color="7" fill="1" visible="yes" active="no"/>
-<layer number="26" name="bNames" color="7" fill="1" visible="yes" active="no"/>
-<layer number="27" name="tValues" color="7" fill="1" visible="yes" active="no"/>
-<layer number="28" name="bValues" color="7" fill="1" visible="yes" active="no"/>
+<layer number="1" name="Top" color="4" fill="1" visible="no" active="no"/>
+<layer number="2" name="Route2" color="16" fill="1" visible="no" active="no"/>
+<layer number="3" name="Route3" color="17" fill="1" visible="no" active="no"/>
+<layer number="4" name="Route4" color="18" fill="1" visible="no" active="no"/>
+<layer number="5" name="Route5" color="19" fill="1" visible="no" active="no"/>
+<layer number="6" name="Route6" color="25" fill="1" visible="no" active="no"/>
+<layer number="7" name="Route7" color="26" fill="1" visible="no" active="no"/>
+<layer number="8" name="Route8" color="27" fill="1" visible="no" active="no"/>
+<layer number="9" name="Route9" color="28" fill="1" visible="no" active="no"/>
+<layer number="10" name="Route10" color="29" fill="1" visible="no" active="no"/>
+<layer number="11" name="Route11" color="30" fill="1" visible="no" active="no"/>
+<layer number="12" name="Route12" color="20" fill="1" visible="no" active="no"/>
+<layer number="13" name="Route13" color="21" fill="1" visible="no" active="no"/>
+<layer number="14" name="Route14" color="22" fill="1" visible="no" active="no"/>
+<layer number="15" name="Route15" color="23" fill="1" visible="no" active="no"/>
+<layer number="16" name="Bottom" color="1" fill="1" visible="no" active="no"/>
+<layer number="17" name="Pads" color="2" fill="1" visible="no" active="no"/>
+<layer number="18" name="Vias" color="2" fill="1" visible="no" active="no"/>
+<layer number="19" name="Unrouted" color="6" fill="1" visible="no" active="no"/>
+<layer number="20" name="Dimension" color="24" fill="1" visible="no" active="no"/>
+<layer number="21" name="tPlace" color="7" fill="1" visible="no" active="no"/>
+<layer number="22" name="bPlace" color="7" fill="1" visible="no" active="no"/>
+<layer number="23" name="tOrigins" color="15" fill="1" visible="no" active="no"/>
+<layer number="24" name="bOrigins" color="15" fill="1" visible="no" active="no"/>
+<layer number="25" name="tNames" color="7" fill="1" visible="no" active="no"/>
+<layer number="26" name="bNames" color="7" fill="1" visible="no" active="no"/>
+<layer number="27" name="tValues" color="7" fill="1" visible="no" active="no"/>
+<layer number="28" name="bValues" color="7" fill="1" visible="no" active="no"/>
 <layer number="29" name="tStop" color="7" fill="3" visible="no" active="no"/>
 <layer number="30" name="bStop" color="7" fill="6" visible="no" active="no"/>
@@
 <layer number="35" name="tGlue" color="7" fill="4" visible="no" active="no"/>
 <layer number="36" name="bGlue" color="7" fill="5" visible="no" active="no"/>
-<layer number="37" name="tTest" color="7" fill="1" visible="yes" active="no"/>
-<layer number="38" name="bTest" color="7" fill="1" visible="yes" active="no"/>
+<layer number="37" name="tTest" color="7" fill="1" visible="no" active="no"/>
+<layer number="38" name="bTest" color="7" fill="1" visible="no" active="no"/>
 <layer number="39" name="tKeepout" color="4" fill="11" visible="no" active="no"/>
 <layer number="40" name="bKeepout" color="1" fill="11" visible="no" active="no"/>
@@
 <layer number="44" name="Drills" color="7" fill="1" visible="no" active="no"/>
 <layer number="45" name="Holes" color="7" fill="1" visible="no" active="no"/>
-<layer number="46" name="Milling" color="3" fill="1" visible="yes" active="no"/>
-<layer number="47" name="Measures" color="7" fill="1" visible="yes" active="no"/>
-<layer number="48" name="Document" color="7" fill="1" visible="yes" active="no"/>
-<layer number="49" name="Reference" color="7" fill="1" visible="yes" active="no"/>
-<layer number="51" name="tDocu" color="7" fill="1" visible="yes" active="no"/>
-<layer number="52" name="bDocu" color="7" fill="1" visible="yes" active="no"/>
+<layer number="46" name="Milling" color="3" fill="1" visible="no" active="no"/>
+<layer number="47" name="Measures" color="7" fill="1" visible="no" active="no"/>
+<layer number="48" name="Document" color="7" fill="1" visible="no" active="no"/>
+<layer number="49" name="Reference" color="7" fill="1" visible="no" active="no"/>
+<layer number="51" name="tDocu" color="7" fill="1" visible="no" active="no"/>
+<layer number="52" name="bDocu" color="7" fill="1" visible="no" active="no"/>
 <layer number="88" name="SimResults" color="9" fill="1" visible="yes" active="yes"/>
 <layer number="89" name="SimProbes" color="9" fill="1" visible="yes" active="yes"/>
@@
 <part name="GND11" library="supply1" library_urn="urn:adsk.eagle:library:371" deviceset="GND" device=""/>
 <part name="U4" library="MAX4545CAP_" deviceset="MAX4545CAP+" device=""/>
-<part name="U$1" library="diy-modules" deviceset="WEMOS-D1-MINI" device=""/>
+<part name="U$1" library="diy-modules" deviceset="WEMOS-D1-MINI" device="" package3d_urn="urn:adsk.eagle:package:29066244/4"/>
 <part name="GND15" library="supply1" library_urn="urn:adsk.eagle:library:371" deviceset="GND" device=""/>
 <part name="OUT1" library="pinhead" library_urn="urn:adsk.eagle:library:325" deviceset="PINHD-1X2" device="" package3d_urn="urn:adsk.eagle:package:22435/2"/>
@@
 <part name="C17" library="rcl" library_urn="urn:adsk.eagle:library:334" deviceset="C-US" device="C0805" package3d_urn="urn:adsk.eagle:package:23617/2" value="100nF"/>
 <part name="GND25" library="supply1" library_urn="urn:adsk.eagle:library:371" deviceset="GND" device=""/>
-<part name="U6" library="LM1117IMP-5.0-NOPB" deviceset="LM1117IMP-5.0-NOPB" device=""/>
+<part name="U6" library="LM1117IMP-5.0-NOPB" deviceset="LM1117IMP-5.0-NOPB" device="" package3d_urn="urn:adsk.eagle:package:29066744/2"/>
 <part name="GND26" library="supply1" library_urn="urn:adsk.eagle:library:371" deviceset="GND" device=""/>
 <part name="C19" library="rcl" library_urn="urn:adsk.eagle:library:334" deviceset="CPOL-EU" device="D/7343-31W" package3d_urn="urn:adsk.eagle:package:23414/2" value="10uF"/>
@@
 <net name="BPOUT2" class="0">
 <segment>
-<pinref part="U$1" gate="G$1" pin="D3"/>
-<wire x1="208.28" y1="271.78" x2="228.6" y2="271.78" width="0.1524" layer="91"/>
-<label x="218.44" y="271.78" size="1.778" layer="95"/>
-</segment>
-<segment>
 <wire x1="106.68" y1="193.04" x2="116.84" y2="193.04" width="0.1524" layer="91"/>
 <pinref part="C1" gate="G$1" pin="1"/>
@@
 <pinref part="U2" gate="G$1" pin="BPOUT"/>
 </segment>
+<segment>
+<pinref part="U$1" gate="G$1" pin="D7"/>
+<wire x1="172.72" y1="269.24" x2="154.94" y2="269.24" width="0.1524" layer="91"/>
+<label x="154.94" y="269.24" size="1.778" layer="95"/>
+</segment>
 </net>
